File: _autosave-DOMO70.sch (KiCad schematic (older format))
At the start: 163 parts, among them SW1 Rotary_Encoder_Switch, SW2 Rotary_Encoder_Switch, U1 AST1109MLTRQ, U2 proton_c, U3 OLED-SSD1306-OLED-SSD1306-4pi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

Commit message: Added routing
Parts:
- added U3: AST1109MLTRQ, Buzzer_Beeper:Buzzer_Mallory_AST1109MLTRQ, symbol Buzzer_AST1109MLTRQ:AST1109MLTRQ
- MX59, MX60, MX61, MX63, MX64, MX65, MX66: footprint MX_Only:MXOnly-1U-NoLED -> MX_Only:MXOnly-1.25U-NoLED
- MX62: footprint MX_Only:MXOnly-1U-NoLED -> MX_Only:MXOnly-6.25U-ReversedStabilizers-NoLED
- MX_29: footprint MX_Only:MXOnly-ISO-ROTATED-ReversedStabilizers-NoLED -> MX_Only:MXOnly-ISO-ReversedStabilizers
- MX_56: footprint (none) -> MX_Only:MXOnly-1.75U-NoLED
- MX_59, MX_61, MX_64, MX_66: footprint MX_Only:MXOnly-1U-NoLED -> MX_Only:MXOnly-1.5U-NoLED
- MX_62: footprint MX_Only:MXOnly-1U-NoLED -> MX_Only:MXOnly-7U-ReversedStabilizers-NoLED
- renumbered U2 to U1, U3 to U2, U1 to U4
Connections:
- net COL8: now also MX67.1 (COL)
- net COL9: now also MX68.1 (COL)
- net GND: now also U3.2 (GND)
- net SPK: now also U3.1 (SPK)
Other:
- moved on the sheet: U4
Changed lines of the file:
@@
 $EndComp
 $Comp
-L proton_c:proton_c U2
+L proton_c:proton_c U1
 U 1 1 5DFDC68C
 P 2550 6000
-F 0 "U2" H 2525 4477 50  0000 C CNN
+F 0 "U1" H 2525 4477 50  0000 C CNN
 F 1 "proton_c" H 2525 4386 50  0000 C CNN
 F 2 "proton_c:proton_c" H 2400 6000 50  0001 C CNN
@@
 $EndComp
 $Comp
-L OLED-SSD1306-4pin-128x32:OLED-SSD1306-OLED-SSD1306-4pin-128x32 U3
+L OLED-SSD1306-4pin-128x32:OLED-SSD1306-OLED-SSD1306-4pin-128x32 U2
 U 1 1 5DFD98F6
 P 5700 6800
-F 0 "U3" H 5617 7175 50  0000 C CNN
+F 0 "U2" H 5617 7175 50  0000 C CNN
 F 1 "OLED-SSD1306-OLED-SSD1306-4pin-128x32" H 5617 7084 50  0000 C CNN
 F 2 "OLED-SSD1306-4pin-128x32:OLED-1306-Supports" H 5700 7200 50  0001 C CNN
@@
 F 0 "MX59" H 1333 4323 60  0000 C CNN
 F 1 "MX-NoLED" H 1333 4249 20  0000 C CNN
-F 2 "MX_Only:MXOnly-1U-NoLED" H 675 4075 60  0001 C CNN
+F 2 "MX_Only:MXOnly-1.25U-NoLED" H 675 4075 60  0001 C CNN
 F 3 "" H 675 4075 60  0001 C CNN
 	1    1300 4100
@@
 F 0 "MX60" H 1783 4323 60  0000 C CNN
 F 1 "MX-NoLED" H 1783 4249 20  0000 C CNN
-F 2 "MX_Only:MXOnly-1U-NoLED" H 1125 4075 60  0001 C CNN
+F 2 "MX_Only:MXOnly-1.25U-NoLED" H 1125 4075 60  0001 C CNN
 F 3 "" H 1125 4075 60  0001 C CNN
 	1    1750 4100
@@
 F 0 "MX61" H 2233 4323 60  0000 C CNN
 F 1 "MX-NoLED" H 2233 4249 20  0000 C CNN
-F 2 "MX_Only:MXOnly-1U-NoLED" H 1575 4075 60  0001 C CNN
+F 2 "MX_Only:MXOnly-1.25U-NoLED" H 1575 4075 60  0001 C CNN
 F 3 "" H 1575 4075 60  0001 C CNN
 	1    2200 4100
@@
 F 0 "MX62" H 2683 4323 60  0000 C CNN
 F 1 "MX-NoLED" H 2683 4249 20  0000 C CNN
-F 2 "MX_Only:MXOnly-1U-NoLED" H 2025 4075 60  0001 C CNN
+F 2 "MX_Only:MXOnly-6.25U-ReversedStabilizers-NoLED" H 2025 4075 60  0001 C CNN
 F 3 "" H 2025 4075 60  0001 C CNN
 	1    2650 4100
@@
 F 0 "MX64" H 3583 4323 60  0000 C CNN
 F 1 "MX-NoLED" H 3583 4249 20  0000 C CNN
-F 2 "MX_Only:MXOnly-1U-NoLED" H 2925 4075 60  0001 C CNN
+F 2 "MX_Only:MXOnly-1.25U-NoLED" H 2925 4075 60  0001 C CNN
 F 3 "" H 2925 4075 60  0001 C CNN
 	1    3550 4100
@@
 F 0 "MX65" H 4033 4323 60  0000 C CNN
 F 1 "MX-NoLED" H 4033 4249 20  0000 C CNN
-F 2 "MX_Only:MXOnly-1U-NoLED" H 3375 4075 60  0001 C CNN
+F 2 "MX_Only:MXOnly-1.25U-NoLED" H 3375 4075 60  0001 C CNN
 F 3 "" H 3375 4075 60  0001 C CNN
 	1    4000 4100
@@
 F 0 "MX63" H 3133 4323 60  0000 C CNN
 F 1 "MX-NoLED" H 3133 4249 20  0000 C CNN
-F 2 "MX_Only:MXOnly-1U-NoLED" H 2475 4075 60  0001 C CNN
+F 2 "MX_Only:MXOnly-1.25U-NoLED" H 2475 4075 60  0001 C CNN
 F 3 "" H 2475 4075 60  0001 C CNN
 	1    3100 4100
@@
 F 0 "MX66" H 4483 4323 60  0000 C CNN
 F 1 "MX-NoLED" H 4483 4249 20  0000 C CNN
-F 2 "MX_Only:MXOnly-1U-NoLED" H 3825 4075 60  0001 C CNN
+F 2 "MX_Only:MXOnly-1.25U-NoLED" H 3825 4075 60  0001 C CNN
 F 3 "" H 3825 4075 60  0001 C CNN
 	1    4450 4100
@@
 Connection ~ 7750 1050
 $Comp
-L Buzzer_AST1109MLTRQ:AST1109MLTRQ U1
+L Buzzer_AST1109MLTRQ:AST1109MLTRQ U4
 U 1 1 5F1A4424
-P 5650 5650
-F 0 "U1" H 5650 5925 50  0000 C CNN
-F 1 "AST1109MLTRQ" H 5650 5834 50  0000 C CNN
-F 2 "Buzzer_Beeper:Buzzer_Mallory_AST1109MLTRQ" H 5650 5650 50  0001 C CNN
-F 3 "" H 5650 5650 50  0001 C CNN
-	1    5650 5650
+P 5600 5550
+F 0 "U4" H 5600 5825 50  0000 C CNN
+F 1 "AST1109MLTRQ" H 5600 5734 50  0000 C CNN
+F 2 "Buzzer_Beeper:Buzzer_Mallory_AST1109MLTRQ" H 5600 5550 50  0001 C CNN
+F 3 "" H 5600 5550 50  0001 C CNN
+	1    5600 5550
 	1    0    0    -1
 $EndComp
@@
 L power:GND #PWR07
 U 1 1 5F1A5FE2
-P 5950 5700
-F 0 "#PWR07" H 5950 5450 50  0001 C CNN
-F 1 "GND" V 5955 5572 50  0000 R CNN
-F 2 "" H 5950 5700 50  0001 C CNN
-F 3 "" H 5950 5700 50  0001 C CNN
-	1    5950 5700
-	0    -1   -1   0
-$EndComp
-Text GLabel 5350 5600 0    50   Input ~ 0
+P 5900 5600
+F 0 "#PWR07" H 5900 5350 50  0001 C CNN
+F 1 "GND" V 5905 5472 50  0000 R CNN
+F 2 "" H 5900 5600 50  0001 C CNN
+F 3 "" H 5900 5600 50  0001 C CNN
+	1    5900 5600
+	0    -1   -1   0
+$EndComp
+Text GLabel 5300 5500 0    50   Input ~ 0
 SPK
 Text GLabel 1500 6900 0    50   Input ~ 0
@@
 F 0 "MX_59" H 1278 4377 50  0000 C CNN
 F 1 "ExtraMX" H 1278 4310 20  0000 C CNN
-F 2 "MX_Only:MXOnly-1U-NoLED" H 1300 4100 50  0001 C CNN
+F 2 "MX_Only:MXOnly-1.5U-NoLED" H 1300 4100 50  0001 C CNN
 F 3 "" H 1300 4100 50  0001 C CNN
 	1    1300 4100
@@
 F 0 "MX_61" H 2178 4377 50  0000 C CNN
 F 1 "ExtraMX" H 2178 4310 20  0000 C CNN
-F 2 "MX_Only:MXOnly-1U-NoLED" H 2200 4100 50  0001 C CNN
+F 2 "MX_Only:MXOnly-1.5U-NoLED" H 2200 4100 50  0001 C CNN
 F 3 "" H 2200 4100 50  0001 C CNN
 	1    2200 4100
@@
 F 0 "MX_62" H 2628 4377 50  0000 C CNN
 F 1 "ExtraMX" H 2628 4310 20  0000 C CNN
-F 2 "MX_Only:MXOnly-1U-NoLED" H 2650 4100 50  0001 C CNN
+F 2 "MX_Only:MXOnly-7U-ReversedStabilizers-NoLED" H 2650 4100 50  0001 C CNN
 F 3 "" H 2650 4100 50  0001 C CNN
 	1    2650 4100
@@
 F 0 "MX_29" H 7128 2127 50  0000 C CNN
 F 1 "ExtraMX" H 7128 2060 20  0000 C CNN
-F 2 "MX_Only:MXOnly-ISO-ROTATED-ReversedStabilizers-NoLED" H 7150 1850 50  0001 C CNN
+F 2 "MX_Only:MXOnly-ISO-ReversedStabilizers" H 7150 1850 50  0001 C CNN
 F 3 "" H 7150 1850 50  0001 C CNN
 	1    7150 1850
@@
 F 0 "MX_64" H 3528 4377 50  0000 C CNN
 F 1 "ExtraMX" H 3528 4310 20  0000 C CNN
-F 2 "MX_Only:MXOnly-1U-NoLED" H 3550 4100 50  0001 C CNN
+F 2 "MX_Only:MXOnly-1.5U-NoLED" H 3550 4100 50  0001 C CNN
 F 3 "" H 3550 4100 50  0001 C CNN
 	1    3550 4100
@@
 F 0 "MX_66" H 4428 4377 50  0000 C CNN
 F 1 "ExtraMX" H 4428 4310 20  0000 C CNN
-F 2 "MX_Only:MXOnly-1U-NoLED" H 4450 4100 50  0001 C CNN
+F 2 "MX_Only:MXOnly-1.5U-NoLED" H 4450 4100 50  0001 C CNN
 F 3 "" H 4450 4100 50  0001 C CNN
 	1    4450 4100
@@
 F 0 "MX_56" H 6228 3627 50  0000 C CNN
 F 1 "ExtraMX" H 6228 3560 20  0000 C CNN
-F 2 "" H 6250 3350 50  0001 C CNN
+F 2 "MX_Only:MXOnly-1.75U-NoLED" H 6250 3350 50  0001 C CNN
 F 3 "" H 6250 3350 50  0001 C CNN
 	1    6250 3350
@@
 Wire Wire Line
 	6150 3500 6200 3500
+Wire Wire Line
+	5050 3300 5050 4050
+Connection ~ 5050 3300
+Wire Wire Line
+	5500 3300 5500 4050
+Connection ~ 5500 3300
+$Comp
+L Buzzer_AST1109MLTRQ:AST1109MLTRQ U3
+U 1 1 5FA1957D
+P 5600 6000
+F 0 "U3" H 5600 6275 50  0000 C CNN
+F 1 "AST1109MLTRQ" H 5600 6184 50  0000 C CNN
+F 2 "Buzzer_Beeper:Buzzer_Mallory_AST1109MLTRQ" H 5600 6000 50  0001 C CNN
+F 3 "" H 5600 6000 50  0001 C CNN
+	1    5600 6000
+	1    0    0    -1
+$EndComp
+$Comp
+L power:GND #PWR0101
+U 1 1 5FA19583
+P 5900 6050
+F 0 "#PWR0101" H 5900 5800 50  0001 C CNN
+F 1 "GND" V 5905 5922 50  0000 R CNN
+F 2 "" H 5900 6050 50  0001 C CNN
+F 3 "" H 5900 6050 50  0001 C CNN
+	1    5900 6050
+	0    -1   -1   0
+$EndComp
+Text GLabel 5300 5950 0    50   Input ~ 0
+SPK
 $EndSCHEMATC
