File: DOMO70.sch (KiCad schematic (older format))
At the start: 163 parts, among them SW1 Rotary_Encoder_Switch, SW2 Rotary_Encoder_Switch, U1 AST1109MLTRQ, U2 proton_c, U3 OLED-SSD1306-OLED-SSD1306-4pi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

Commit message: Updating who-knows-what
Parts:
- added U3: AST1109MLTRQ, Buzzer_Beeper:Buzzer_Mallory_AST1109MLTRQ, symbol Buzzer_AST1109MLTRQ:AST1109MLTRQ
- MX_29: footprint MX_Only:MXOnly-ISO-ROTATED-ReversedStabilizers-NoLED -> MX_Only:MXOnly-ISO-ReversedStabilizers
- renumbered U2 to U1, U3 to U2, U1 to U4
Connections:
- net COL8: now also MX67.1 (COL)
- net COL9: now also MX68.1 (COL)
- net GND: now also U3.2 (GND)
- net SPK: now also U3.1 (SPK)
Other:
- moved on the sheet: U4
Changed lines of the file:
@@
 $EndComp
 $Comp
-L proton_c:proton_c U2
+L proton_c:proton_c U1
 U 1 1 5DFDC68C
 P 2550 6000
-F 0 "U2" H 2525 4477 50  0000 C CNN
+F 0 "U1" H 2525 4477 50  0000 C CNN
 F 1 "proton_c" H 2525 4386 50  0000 C CNN
 F 2 "proton_c:proton_c" H 2400 6000 50  0001 C CNN
@@
 $EndComp
 $Comp
-L OLED-SSD1306-4pin-128x32:OLED-SSD1306-OLED-SSD1306-4pin-128x32 U3
+L OLED-SSD1306-4pin-128x32:OLED-SSD1306-OLED-SSD1306-4pin-128x32 U2
 U 1 1 5DFD98F6
 P 5700 6800
-F 0 "U3" H 5617 7175 50  0000 C CNN
+F 0 "U2" H 5617 7175 50  0000 C CNN
 F 1 "OLED-SSD1306-OLED-SSD1306-4pin-128x32" H 5617 7084 50  0000 C CNN
 F 2 "OLED-SSD1306-4pin-128x32:OLED-1306-Supports" H 5700 7200 50  0001 C CNN
@@
 Connection ~ 7750 1050
 $Comp
-L Buzzer_AST1109MLTRQ:AST1109MLTRQ U1
+L Buzzer_AST1109MLTRQ:AST1109MLTRQ U4
 U 1 1 5F1A4424
-P 5650 5650
-F 0 "U1" H 5650 5925 50  0000 C CNN
-F 1 "AST1109MLTRQ" H 5650 5834 50  0000 C CNN
-F 2 "Buzzer_Beeper:Buzzer_Mallory_AST1109MLTRQ" H 5650 5650 50  0001 C CNN
-F 3 "" H 5650 5650 50  0001 C CNN
-	1    5650 5650
+P 5600 5550
+F 0 "U4" H 5600 5825 50  0000 C CNN
+F 1 "AST1109MLTRQ" H 5600 5734 50  0000 C CNN
+F 2 "Buzzer_Beeper:Buzzer_Mallory_AST1109MLTRQ" H 5600 5550 50  0001 C CNN
+F 3 "" H 5600 5550 50  0001 C CNN
+	1    5600 5550
 	1    0    0    -1
 $EndComp
@@
 L power:GND #PWR07
 U 1 1 5F1A5FE2
-P 5950 5700
-F 0 "#PWR07" H 5950 5450 50  0001 C CNN
-F 1 "GND" V 5955 5572 50  0000 R CNN
-F 2 "" H 5950 5700 50  0001 C CNN
-F 3 "" H 5950 5700 50  0001 C CNN
-	1    5950 5700
-	0    -1   -1   0
-$EndComp
-Text GLabel 5350 5600 0    50   Input ~ 0
+P 5900 5600
+F 0 "#PWR07" H 5900 5350 50  0001 C CNN
+F 1 "GND" V 5905 5472 50  0000 R CNN
+F 2 "" H 5900 5600 50  0001 C CNN
+F 3 "" H 5900 5600 50  0001 C CNN
+	1    5900 5600
+	0    -1   -1   0
+$EndComp
+Text GLabel 5300 5500 0    50   Input ~ 0
 SPK
 Text GLabel 1500 6900 0    50   Input ~ 0
@@
 F 0 "MX_29" H 7128 2127 50  0000 C CNN
 F 1 "ExtraMX" H 7128 2060 20  0000 C CNN
-F 2 "MX_Only:MXOnly-ISO-ROTATED-ReversedStabilizers-NoLED" H 7150 1850 50  0001 C CNN
+F 2 "MX_Only:MXOnly-ISO-ReversedStabilizers" H 7150 1850 50  0001 C CNN
 F 3 "" H 7150 1850 50  0001 C CNN
 	1    7150 1850
@@
 Wire Wire Line
 	6150 3500 6200 3500
+Wire Wire Line
+	5050 3300 5050 4050
+Connection ~ 5050 3300
+Wire Wire Line
+	5500 3300 5500 4050
+Connection ~ 5500 3300
+$Comp
+L Buzzer_AST1109MLTRQ:AST1109MLTRQ U3
+U 1 1 5FA1957D
+P 5600 6000
+F 0 "U3" H 5600 6275 50  0000 C CNN
+F 1 "AST1109MLTRQ" H 5600 6184 50  0000 C CNN
+F 2 "Buzzer_Beeper:Buzzer_Mallory_AST1109MLTRQ" H 5600 6000 50  0001 C CNN
+F 3 "" H 5600 6000 50  0001 C CNN
+	1    5600 6000
+	1    0    0    -1
+$EndComp
+$Comp
+L power:GND #PWR0101
+U 1 1 5FA19583
+P 5900 6050
+F 0 "#PWR0101" H 5900 5800 50  0001 C CNN
+F 1 "GND" V 5905 5922 50  0000 R CNN
+F 2 "" H 5900 6050 50  0001 C CNN
+F 3 "" H 5900 6050 50  0001 C CNN
+	1    5900 6050
+	0    -1   -1   0
+$EndComp
+Text GLabel 5300 5950 0    50   Input ~ 0
+SPK
 $EndSCHEMATC

Commit message: Added routes, graphics
Parts:
- D1, D10, D11, D12, D13, D14, D15, D16, D17, D18, D19, D2, D20, D21, D22, D23, D24, D25, D26, D27, D28, D29, D3, D30, D31, D32, D33, D34, D35, D36, D37, D38, D39, D4, D40, D41, D42, D43, D44, D45, D46, D47, D48, D49, D5, D50, D51, D52, D53, D54, D55, D56, D57, D58, D59, D6, D60, D61, D62, D63, D64, D65, D66, D67, D68, D69, D7, D70, D71, D72, D8, D9, DE1, DE2: symbol Diode:1N4148 -> DOMO70-rescue:1N4148-Diode
- MX1, MX10, MX11, MX12, MX13, MX14, MX15, MX16, MX17, MX18, MX19, MX2, MX20, MX21, MX22, MX23, MX24, MX25, MX26, MX27, MX28, MX29, MX3, MX30, MX31, MX32, MX33, MX34, MX35, MX36, MX37, MX38, MX39, MX4, MX40, MX41, MX42, MX43, MX44, MX45, MX46, MX47, MX48, MX49, MX5, MX50, MX51, MX52, MX53, MX54, MX55, MX56, MX57, MX58, MX59, MX6, MX60, MX61, MX62, MX63, MX64, MX65, MX66, MX67, MX68, MX69, MX7, MX70, MX71, MX72, MX8, MX9: symbol MX_Alps_Hybrid:MX-NoLED -> DOMO70-rescue:MX-NoLED-MX_Alps_Hybrid
- SW1, SW2: symbol Device:Rotary_Encoder_Switch -> DOMO70-rescue:Rotary_Encoder_Switch-Device
- U1: symbol proton_c:proton_c -> DOMO70-rescue:proton_c-proton_c
Connections:
- no-connect marks 5 -> 15
